File: pcb_mainboard/pcb_mainboard.kicad_sch (KiCad schematic)
At the start: 10 parts, among them J1 Ringer Module, J2 Phone Body, Q1 Q_NMOS_GSD, Q2 Q_NMOS_GSD, U1 Adafruit_Audio_FX_+_Amp

Commit message: V1 board as sent to oshpark
Parts:
- Q1, Q2: footprint Package_TO_SOT_SMD:SOT-416 -> Package_TO_SOT_THT:TO-251-3-1EP_Horizontal_TabDown
- renumbered BT1 to 9V1, U1 to A1, A1 to A2
Connections:
- net GND: now also J2.2 (Pin_2); no longer J2.4 (Pin_4)
- net SW_DIAL: now also J2.3 (Pin_3); no longer J2.2 (Pin_2)
- net SW_HOOK: now also J2.4 (Pin_4); no longer J2.3 (Pin_3)
